Commit message: refactoring for new file structure

File: robot_models/turtlebot3_description/urdf/turtlebot3_burger_for_lane_recognition.urdf.xacro (robot description, xacro)
@@ -176,5 +176,5 @@
       <origin xyz="0 0 0" rpy="0 0 0"/>
       <geometry>
-        <box size="0.17 0.19 0.05"/>
+        <box size="0.11 0.19 0.05"/>
       </geometry>
     </collision>
